File: Platine/HB-UNI-Sen-Lev-Vo.kicad_pcb (KiCad board)
At the start: 2 copper layers, 55.9 x 53.3 mm, 17 parts, among them J1 12V DC, J2 D24V5F5, J6 Sonde, J8 PROG, SW1 CONFIG_BUTTON, U1 ArduinoProMini, U2 CC1101

Commit message: Images PCB
Parts:
- Copy: value Version 1.0.2 - 03/2019 -> Version 1.0.3 - 02/2020
Other:
- board text added: "HB-UNI-Sen-Lev-Vo"
- board text removed: "HB-Sen-MULTI"
Changed lines of the file:
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@@
   (page A4)
   (title_block
-    (title HB-Sen-Multi)
+    (title HB-UNI-Sen-Lev-Vo)
     (date 2019-03-11)
-    (rev V1.0.2)
+    (rev V1.0.3)
     (comment 1 "© Silvio Sternitzke")
-    (comment 2 "Multi Sensoren PBC")
+    (comment 2 "Sensoren PBC - Votronic-Sonden")
   )
   (layers
@@
       (effects (font (size 1.2 1.2) (thickness 0.12)))
     )
-    (fp_text value "Version 1.0.2 - 03/2019" (at -2.4003 -1.9939 90) (layer B.SilkS)
+    (fp_text value "Version 1.0.3 - 02/2020" (at -2.4003 -1.7399 90) (layer B.SilkS)
       (effects (font (size 0.9 0.75) (thickness 0.12)) (justify mirror))
     )
@@
     (effects (font (size 1.5 1.5) (thickness 0.3)))
   )
-  (gr_text HB-Sen-MULTI (at 175.26 83.185 90) (layer B.SilkS)
+  (gr_text HB-UNI-Sen-Lev-Vo (at 175.26 85.09 90) (layer B.SilkS)
     (effects (font (size 0.9 0.75) (thickness 0.1875)) (justify mirror))
   )

Commit message: readme.md
Parts:
- SW1: value CONFIG_BUTTON -> CONFIG
Changed lines of the file:
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@@
       (effects (font (size 1 1) (thickness 0.15)))
     )
-    (fp_text value 10uF (at 0.75 3.25 90) (layer F.Fab)
+    (fp_text value 10uF (at 0.75 2.858 90) (layer F.SilkS)
       (effects (font (size 1 1) (thickness 0.15)))
     )
@@
     (descr "LED, diameter 3.0mm, 2 pins")
     (tags "LED diameter 3.0mm 2 pins")
-    (fp_text reference D1 (at 1.27 -2.96 270) (layer F.SilkS)
-      (effects (font (size 1 1) (thickness 0.15)))
-    )
-    (fp_text value LED (at 1.27 2.96 270) (layer F.Fab)
+    (fp_text reference D1 (at 2.9845 -2.54 270) (layer F.SilkS)
+      (effects (font (size 1 1) (thickness 0.15)))
+    )
+    (fp_text value LED (at -0.0635 -2.667 270) (layer F.SilkS)
       (effects (font (size 1 1) (thickness 0.15)))
     )
@@
     (descr "Through hole straight pin header, 1x06, 2.54mm pitch, single row")
     (tags "Through hole pin header THT 1x06 2.54mm single row")
-    (fp_text reference J8 (at 0 -2.33) (layer F.SilkS)
-      (effects (font (size 1 1) (thickness 0.15)))
-    )
-    (fp_text value PROG (at 0 15.03) (layer F.Fab)
+    (fp_text reference J8 (at -0.508 -2.54) (layer F.SilkS)
+      (effects (font (size 1 1) (thickness 0.15)))
+    )
+    (fp_text value PROG (at 0 15.367) (layer F.SilkS)
       (effects (font (size 1 1) (thickness 0.15)))
     )
@@
     (descr "Resistor, Axial_DIN0207 series, Axial, Vertical, pin pitch=2.54mm, 0.25W = 1/4W, length*diameter=6.3*2.5mm^2, http://cdn-reichelt.de/documents/datenblatt/B400/1_4W%23YAG.pdf")
     (tags "Resistor Axial_DIN0207 series Axial Vertical pin pitch 2.54mm 0.25W = 1/4W length 6.3mm diameter 2.5mm")
-    (fp_text reference R1 (at 1.27 -2.37 270) (layer F.SilkS)
-      (effects (font (size 1 1) (thickness 0.15)))
-    )
-    (fp_text value 330 (at 1.27 2.37 270) (layer F.Fab)
+    (fp_text reference R1 (at 4.572 0.127 270) (layer F.SilkS)
+      (effects (font (size 1 1) (thickness 0.15)))
+    )
+    (fp_text value 330 (at 1.016 -2.286 270) (layer F.SilkS)
       (effects (font (size 1 1) (thickness 0.15)))
     )
@@
     (fp_line (start 3.59 1.5) (end 3.59 -1.5) (layer F.CrtYd) (width 0.05))
     (fp_line (start 3.59 -1.5) (end -1.5 -1.5) (layer F.CrtYd) (width 0.05))
-    (fp_text user %R (at 1.27 -2.37 270) (layer F.Fab)
+    (fp_text user %R (at 4.572 0.127 270) (layer F.Fab)
       (effects (font (size 1 1) (thickness 0.15)))
     )
@@
     (descr "tactile push button, 6x6mm e.g. PHAP33xx series, height=5mm")
     (tags "tact sw push 6mm")
-    (fp_text reference SW1 (at 3.25 -2 180) (layer F.SilkS)
-      (effects (font (size 1 1) (thickness 0.15)))
-    )
-    (fp_text value CONFIG_BUTTON (at 3.75 6.7 180) (layer F.Fab)
-      (effects (font (size 1 1) (thickness 0.15)))
-    )
-    (fp_text user %R (at 3.25 2.25 180) (layer F.Fab)
+    (fp_text reference SW1 (at 3.25 2.2225 180) (layer F.Fab)
+      (effects (font (size 1 1) (thickness 0.15)))
+    )
+    (fp_text value CONFIG (at 2.667 6.7 180) (layer F.SilkS)
+      (effects (font (size 1 1) (thickness 0.15)))
+    )
+    (fp_text user %R (at 3.25 2.25 180) (layer F.SilkS)
       (effects (font (size 1 1) (thickness 0.15)))
     )
@@
   (module Homebrew:ArduinoProMini (layer F.Cu)
     (at 171.45 83.82 90)
-    (fp_text reference U1 (at 3.81 -13.97 90) (layer F.SilkS) hide
-      (effects (font (size 1 1) (thickness 0.15)))
-    )
-    (fp_text value ArduinoProMini (at 16.51 -8.89 90) (layer F.Fab)
+    (fp_text reference U1 (at 1.397 -13.081 90) (layer F.SilkS) hide
+      (effects (font (size 1 1) (thickness 0.15)))
+    )
+    (fp_text value ArduinoProMini (at 16.51 -8.89 90) (layer F.SilkS)
       (effects (font (size 1 1) (thickness 0.15)))
     )
@@
       (effects (font (size 1 1) (thickness 0.15)))
     )
-    (fp_text value CC1101 (at 15.5 15) (layer F.Fab)
+    (fp_text value CC1101 (at 11.176 8.128) (layer F.SilkS)
       (effects (font (size 1 1) (thickness 0.15)))
     )
@@
     (descr "Through hole straight pin header, 1x04, 2.54mm pitch, single row")
     (tags "Through hole pin header THT 1x04 2.54mm single row")
-    (fp_text reference J2 (at 0 -2.33 180) (layer F.SilkS)
-      (effects (font (size 1 1) (thickness 0.15)))
-    )
-    (fp_text value D24V5F5 (at 0 9.95 180) (layer F.Fab)
+    (fp_text reference J2 (at 0 -2.794 180) (layer F.SilkS)
+      (effects (font (size 1 1) (thickness 0.15)))
+    )
+    (fp_text value D24V5F5 (at 2.984 3.556 270) (layer F.SilkS)
       (effects (font (size 1 1) (thickness 0.15)))
     )
@@
       (effects (font (size 1 1) (thickness 0.15)))
     )
-    (fp_text value "12V DC" (at 2.2225 6.0325 90) (layer F.SilkS)
+    (fp_text value "12V DC" (at 2.2225 5.334 90) (layer F.SilkS)
       (effects (font (size 1 1) (thickness 0.15)))
     )
@@
       (effects (font (size 1 1) (thickness 0.15)))
     )
-    (fp_text value Sonde (at 14.732 1.778 180) (layer F.SilkS)
-      (effects (font (size 1 1) (thickness 0.15)))
-    )
+    (fp_text value Sonde (at -5.334 -8.065 180) (layer F.SilkS)
+      (effects (font (size 1 1) (thickness 0.15)))
+    )
